File: KiCAD/remoteboy.kicad_sch (KiCad schematic)
At the start: 36 parts, among them Q1 MMBT2222A, SW1 SW_Push, SW10 SW_Push, SW2 SW_Push, SW3 SW_Push, SW4 SW_Push, SW5 SW_Push, SW6 SW_Push, SW7 SW_Push, SW8 SW_Push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

Commit message: Fix schematic and pcb
Parts:
- R5, R6: value 470 -> 220
Connections:
- net ROW1: now also D4.2 (A), D9.2 (A); no longer D4.1 (K), D9.1 (K)
- net ROW2: now also D10.2 (A), D5.2 (A); no longer D10.1 (K), D5.1 (K)
- net ROW3: now also D11.2 (A), D6.2 (A); no longer D11.1 (K), D6.1 (K)
- net ROW4: now also D12.2 (A), D7.2 (A); no longer D12.1 (K), D7.1 (K)
- net ROW5: now also D13.2 (A), D8.2 (A); no longer D13.1 (K), D8.1 (K)
- net at SW2.1: now also D5.1 (K); no longer D5.2 (A)
- net at SW7.1: now also D10.1 (K); no longer D10.2 (A)
- net at SW1.1: now also D4.1 (K); no longer D4.2 (A)
- net at SW10.1: now also D13.1 (K); no longer D13.2 (A)
- net at SW8.1: now also D11.1 (K); no longer D11.2 (A)
- net at SW6.1: now also D9.1 (K); no longer D9.2 (A)
- net at SW5.1: now also D8.1 (K); no longer D8.2 (A)
- net at SW3.1: now also D6.1 (K); no longer D6.2 (A)
- net at SW4.1: now also D7.1 (K); no longer D7.2 (A)
- net at SW9.1: now also D12.1 (K); no longer D12.2 (A)
Other:
- moved on the sheet: D10, D11, D12, D13, D4, D5, D6, D7, D8, D9
Changed lines of the file:
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@@
 	(wire
 		(pts
+			(xy 134.62 97.79) (xy 162.56 97.79)
+		)
+		(stroke
+			(width 0)
+			(type default)
+		)
+	)
+	(wire
+		(pts
 			(xy 134.62 55.88) (xy 137.16 55.88)
 		)
@@
 	(wire
 		(pts
-			(xy 162.56 85.09) (xy 134.62 85.09)
+			(xy 134.62 59.69) (xy 162.56 59.69)
 		)
 		(stroke
@@
 	(wire
 		(pts
-			(xy 162.56 59.69) (xy 134.62 59.69)
+			(xy 129.54 97.79) (xy 134.62 97.79)
 		)
 		(stroke
@@
 	(wire
 		(pts
-			(xy 129.54 97.79) (xy 134.62 97.79)
+			(xy 101.6 71.12) (xy 101.6 73.66)
 		)
 		(stroke
@@
 	(wire
 		(pts
-			(xy 101.6 71.12) (xy 101.6 73.66)
+			(xy 162.56 55.88) (xy 162.56 59.69)
 		)
 		(stroke
@@
 	(wire
 		(pts
-			(xy 162.56 55.88) (xy 162.56 59.69)
+			(xy 134.62 72.39) (xy 162.56 72.39)
 		)
 		(stroke
@@
 	(wire
 		(pts
-			(xy 162.56 72.39) (xy 134.62 72.39)
-		)
-		(stroke
-			(width 0)
-			(type default)
-		)
-	)
-	(wire
-		(pts
 			(xy 101.6 33.02) (xy 101.6 40.64)
 		)
@@
 	(wire
 		(pts
-			(xy 158.75 43.18) (xy 154.94 43.18)
+			(xy 134.62 46.99) (xy 162.56 46.99)
 		)
 		(stroke
@@
 	(wire
 		(pts
-			(xy 162.56 46.99) (xy 134.62 46.99)
+			(xy 158.75 43.18) (xy 154.94 43.18)
 		)
 		(stroke
@@
 	(wire
 		(pts
-			(xy 162.56 97.79) (xy 134.62 97.79)
+			(xy 134.62 85.09) (xy 162.56 85.09)
 		)
 		(stroke
@@
 	(symbol
 		(lib_id "Diode:1N4148W")
-		(at 140.97 55.88 0)
+		(at 140.97 55.88 180)
 		(unit 1)
 		(exclude_from_sim no)
@@
 		)
 		(property "Footprint" "Diode_SMD:D_SOD-123"
-			(at 140.97 60.325 0)
+			(at 140.97 51.435 0)
 			(effects
 				(font
@@
 	(symbol
 		(lib_id "Diode:1N4148W")
-		(at 166.37 93.98 0)
+		(at 166.37 93.98 180)
 		(unit 1)
 		(exclude_from_sim no)
@@
 		)
 		(property "Footprint" "Diode_SMD:D_SOD-123"
-			(at 166.37 98.425 0)
+			(at 166.37 89.535 0)
 			(effects
 				(font
@@
 			)
 		)
-		(property "Value" "470"
+		(property "Value" "220"
 			(at 55.88 95.25 90)
 			(effects
@@
 	(symbol
 		(lib_id "Diode:1N4148W")
-		(at 166.37 55.88 0)
+		(at 166.37 55.88 180)
 		(unit 1)
 		(exclude_from_sim no)
@@
 		)
 		(property "Footprint" "Diode_SMD:D_SOD-123"
-			(at 166.37 60.325 0)
+			(at 166.37 51.435 0)
 			(effects
 				(font
@@
 			)
 		)
-		(property "Value" "470"
+		(property "Value" "220"
 			(at 55.88 113.03 90)
 			(effects
@@
 	(symbol
 		(lib_id "Diode:1N4148W")
-		(at 166.37 43.18 0)
+		(at 166.37 43.18 180)
 		(unit 1)
 		(exclude_from_sim no)
@@
 		)
 		(property "Footprint" "Diode_SMD:D_SOD-123"
-			(at 166.37 47.625 0)
+			(at 166.37 38.735 0)
 			(effects
 				(font
@@
 	(symbol
 		(lib_id "Diode:1N4148W")
-		(at 166.37 68.58 0)
+		(at 166.37 68.58 180)
 		(unit 1)
 		(exclude_from_sim no)
@@
 		)
 		(property "Footprint" "Diode_SMD:D_SOD-123"
-			(at 166.37 73.025 0)
+			(at 166.37 64.135 0)
 			(effects
 				(font
@@
 	(symbol
 		(lib_id "Diode:1N4148W")
-		(at 140.97 81.28 0)
+		(at 140.97 81.28 180)
 		(unit 1)
 		(exclude_from_sim no)
@@
 		)
 		(property "Footprint" "Diode_SMD:D_SOD-123"
-			(at 140.97 85.725 0)
+			(at 140.97 76.835 0)
 			(effects
 				(font
@@
 	(symbol
 		(lib_id "Diode:1N4148W")
-		(at 140.97 43.18 0)
+		(at 140.97 43.18 180)
 		(unit 1)
 		(exclude_from_sim no)
@@
 		)
 		(property "Footprint" "Diode_SMD:D_SOD-123"
-			(at 140.97 47.625 0)
+			(at 140.97 38.735 0)
 			(effects
 				(font
@@
 	(symbol
 		(lib_id "Diode:1N4148W")
-		(at 140.97 93.98 0)
+		(at 140.97 93.98 180)
 		(unit 1)
 		(exclude_from_sim no)
@@
 		)
 		(property "Footprint" "Diode_SMD:D_SOD-123"
-			(at 140.97 98.425 0)
+			(at 140.97 89.535 0)
 			(effects
 				(font
@@
 	(symbol
 		(lib_id "Diode:1N4148W")
-		(at 166.37 81.28 0)
+		(at 166.37 81.28 180)
 		(unit 1)
 		(exclude_from_sim no)
@@
 		)
 		(property "Footprint" "Diode_SMD:D_SOD-123"
-			(at 166.37 85.725 0)
+			(at 166.37 76.835 0)
 			(effects
 				(font
@@
 	(symbol
 		(lib_id "Diode:1N4148W")
-		(at 140.97 68.58 0)
+		(at 140.97 68.58 180)
 		(unit 1)
 		(exclude_from_sim no)
@@
 		)
 		(property "Footprint" "Diode_SMD:D_SOD-123"
-			(at 140.97 73.025 0)
+			(at 140.97 64.135 0)
 			(effects
 				(font
